File: I/2026/minilab/placas/salidas/salidas.kicad_sch (KiCad schematic)
At the start: 26 parts, among them SW1 SW_DPST_x2, SW2 SW_DPST_x2, SW3 SW_DPST_x2, SW4 SW_DPST_x2, SW5 SW_DPST_x2, SW6 SW_DPST_x2

Commit message: check entradas
Parts:
- 5V1, GND1: value ~ -> (none); footprint Library:PinHeader_1x01_P1.00mm_VerticalBIG -> Connector_PinHeader_1.00mm:PinHeader_1x01_P1.00mm_Vertical
- C1, C2, C3, C4, C5, C6: footprint Library:CP_Radial_D5.0mm_P2.00mmBIG -> Capacitor_THT:CP_Radial_D5.0mm_P2.00mm
- R1, R2, R3, R4, R5, R6: footprint Library:R_Axial_DIN0207_L6.3mm_D2.5mm_P7.62mm_HorizontalBIG -> Resistor_THT:R_Axial_DIN0207_L6.3mm_D2.5mm_P7.62mm_Horizontal
- SW1, SW6: footprint Library:SW_DIP_SPSTx01_Slide_9.78x4.72mm_W7.62mm_P2.54mmBIG -> Button_Switch_THT:SW_DIP_SPSTx01_Slide_9.78x4.72mm_W7.62mm_P2.54mm
- SW2: renamed from SW4; footprint Library:SW_DIP_SPSTx01_Slide_9.78x4.72mm_W7.62mm_P2.54mmBIG -> Button_Switch_THT:SW_DIP_SPSTx01_Slide_9.78x4.72mm_W7.62mm_P2.54mm
- SW3: renamed from SW2; footprint Library:SW_DIP_SPSTx01_Slide_9.78x4.72mm_W7.62mm_P2.54mmBIG -> Button_Switch_THT:SW_DIP_SPSTx01_Slide_9.78x4.72mm_W7.62mm_P2.54mm
- SW4: renamed from SW5; footprint Library:SW_DIP_SPSTx01_Slide_9.78x4.72mm_W7.62mm_P2.54mmBIG -> Button_Switch_THT:SW_DIP_SPSTx01_Slide_9.78x4.72mm_W7.62mm_P2.54mm
- SW5: renamed from SW3; footprint Library:SW_DIP_SPSTx01_Slide_9.78x4.72mm_W7.62mm_P2.54mmBIG -> Button_Switch_THT:SW_DIP_SPSTx01_Slide_9.78x4.72mm_W7.62mm_P2.54mm
- TERMINAL1, TERMINAL2, TERMINAL3, TERMINAL4, TERMINAL5, TERMINAL6: footprint Library:PinHeader_1x01_P1.00mm_VerticalBIG -> Connector_PinHeader_1.00mm:PinHeader_1x01_P1.00mm_Vertical
